Commit message: Added Suction Model to Dual Arm

File: wrs_gazebo/mobile_dual_arm/urdf/mobile_dual_arm.xacro (robot description, xacro)
@@ -3,6 +3,7 @@
 	<xacro:include filename="$(find single_arm_description)/urdf/single_arm.xacro" />
 	<xacro:include filename="$(find Slide_rail)/urdf/Slide_rail.xacro" />
+	<xacro:include filename="$(find suction_urdf)/urdf/suction_urdf.xacro" />
 	<!--xacro:include filename="$(find single_arm_description)/urdf/materials.xacro" /-->
-        <xacro:include filename="$(find mobile_dual_arm)/urdf/mobile_dual_arm.gazebo" />
+  <xacro:include filename="$(find mobile_dual_arm)/urdf/mobile_dual_arm.gazebo" />
         <!--xacro:include filename="$(find mobile_table)/urdf/mobile_table.xacro" /-->
 	<link name="world"/>
@@ -21,10 +22,16 @@
      		<child link="mobile_base"/>
 	</joint-->
-        <xacro:single_arm side="r"  parent="Arm_Base_R_Link">
+  <xacro:single_arm side="r"  parent="Arm_Base_R_Link" child="r_tool_link">
 	  <origin xyz="0 -0.016 0" rpy="1.57 1.57 0" />
-        </xacro:single_arm>
-        <xacro:single_arm side="l"  parent="Arm_Base_L_Link">
+  </xacro:single_arm>
+  <xacro:suction side="r"  parent="r_Link_6">
+	  <origin xyz="0 -0.016 0" rpy="0 0 0" />
+  </xacro:suction>
+  <xacro:single_arm side="l"  parent="Arm_Base_L_Link" child="l_tool_link">
 	  <origin xyz="0 0.016 0" rpy="-1.57 1.57 0" />
-        </xacro:single_arm>
+  </xacro:single_arm>
+  <xacro:suction side="l"  parent="l_Link_6">
+	  <origin xyz="0 0.016 0" rpy="0 0 0" />
+  </xacro:suction>
 	<!--joint name="fixed" type="fixed">
 		<origin

File: wrs_gazebo/single_arm/single_arm_description/urdf/single_arm.gazebo.xacro (robot description, xacro)
@@ -54,10 +54,10 @@
     <selfCollide>false</selfCollide>
   </gazebo>
-  <gazebo reference="${side}_Link_7">
+  <!-- <gazebo reference="${side}_Link_7">
     <mu1>0.2</mu1>
     <mu2>0.2</mu2>
     <material>Gazebo/Black</material>
     <selfCollide>false</selfCollide>
-  </gazebo>
+  </gazebo> -->
   <!--
   <gazebo reference="${side}_Link_8">

File: wrs_gazebo/single_arm/single_arm_description/urdf/single_arm.xacro (robot description, xacro)
@@ -5,5 +5,5 @@
   <xacro:include filename="$(find single_arm_description)/urdf/materials.xacro" />
   <!-- Constants for robot dimensions -->
-  <xacro:macro name="single_arm" params="side parent *origin">
+  <xacro:macro name="single_arm" params="side parent child *origin">
 	  <link
 	    name="${side}_Base">
@@ -399,5 +399,5 @@
 	      velocity="5" />
 	  </joint>
-	  <link
+	  <!-- <link
 	    name="${side}_Link_7">
 	    <inertial>
@@ -438,15 +438,15 @@
 	      </geometry>
 	    </collision>
-	  </link>
+	  </link> -->
 	  <joint
 	    name="${side}_joint_7"
 	    type="revolute">
 	    <origin
-	      xyz="0 0 0"
+	      xyz="0 -0.1345 0"
 	      rpy="1.5708 4.5659E-16 1.2025E-31" />
 	    <parent
 	      link="${side}_Link_6" />
 	    <child
-	      link="${side}_Link_7" />
+	      link="${child}" />
 	    <axis
 	      xyz="0 0 1" />

Commit message: Added Vacuum Gripper Plugin & Mobile Table in Gazebo Modle Added New Strategy File

File: wrs_gazebo/mobile_dual_arm/urdf/mobile_dual_arm.xacro (robot description, xacro)
@@ -6,20 +6,20 @@
 	<!--xacro:include filename="$(find single_arm_description)/urdf/materials.xacro" /-->
   <xacro:include filename="$(find mobile_dual_arm)/urdf/mobile_dual_arm.gazebo" />
-        <!--xacro:include filename="$(find mobile_table)/urdf/mobile_table.xacro" /-->
+  <xacro:include filename="$(find mobile_table)/urdf/mobile_table.xacro" />
 	<link name="world"/>
-	<joint name="fixed1" type="fixed">
+	<!-- <joint name="fixed1" type="fixed">
+		<origin
+	    xyz="0 0 0.562"
+      rpy="0 0 0" />
+		<parent link="world"/>
+    <child link="base_link"/>
+	</joint> -->
+	<joint name="fixed3" type="fixed">
 		<origin
 	    	xyz="0 0 0.562"
-        	rpy="0 0 0" />
+        rpy="0 0 0" />
 		<parent link="world"/>
-     		<child link="base_link"/>
+    <child link="mobile_base"/>
 	</joint>
-	<!--joint name="fixed3" type="fixed">
-		<origin
-	    	xyz="0 0 0.562"
-        	rpy="0 0 0" />
-		<parent link="world"/>
-     		<child link="mobile_base"/>
-	</joint-->
   <xacro:single_arm side="r"  parent="Arm_Base_R_Link" child="r_tool_link">
 	  <origin xyz="0 -0.016 0" rpy="1.57 1.57 0" />
@@ -41,11 +41,11 @@
      		<child link="Base"/>
 	</joint-->
-	<!--joint name="fixed1" type="fixed">
+	<joint name="fixed1" type="fixed">
 		<origin
-	    	xyz="0 0 0.1"
-        	rpy="0 0 0" />
+	    xyz="0 0 0"
+      rpy="0 0 0" />
 		<parent link="mobile_base"/>
-     		<child link="base_link"/>
-	</joint-->
+    <child link="base_link"/>
+	</joint>
 	<!--joint name="fixed2" type="fixed">
 		<origin

File: wrs_gazebo/suction_urdf/urdf/suction_urdf.xacro (robot description, xacro)
@@ -102,4 +102,48 @@
         velocity="5" />
     </joint>
+    <link
+      name="${side}_end_Link">
+      <inertial>
+        <origin
+          xyz="0 0 0"
+          rpy="0 0 0" />
+        <mass
+          value="0.000438" />
+        <inertia
+          ixx="2.0813E-05"
+          ixy="1.7379E-08"
+          ixz="9.2823E-08"
+          iyy="1.8619E-05"
+          iyz="4.6462E-06"
+          izz="5.6779E-06" />
+      </inertial>
+      <visual>
+        <origin
+          xyz="0 0 0"
+          rpy="0 0 0" />
+	<geometry>
+           <box size="0.01 0.01 0.01"/>
+        </geometry>
+        <material
+          name="">
+          <color
+            rgba="0.79216 0.81961 0.93333 1" />
+        </material>
+      </visual>
+    </link>
+    <joint name="${side}_end_joint" type="revolute">
+	<origin
+        xyz="0 0 0.09"
+        rpy="-1.7985E-15 -2.9973E-16 1.1669E-16" />
+	<parent link="${side}_tool_end_Link"/>
+	<child link="${side}_end_Link"/>
+        <axis
+            xyz="0 1 0" />
+        <limit
+            lower="-3.14"
+	    upper="3.14"
+            effort="5"
+            velocity="5" />
+    </joint>
     <xacro:suction_transmission side="${side}" />
     <xacro:suction_gazebo side="${side}" />

Commit message: Added Example Task File : example.py Modified DHLink for New Suction Modfied Some  Error in Get Phi Angle

File: wrs_gazebo/mobile_dual_arm/urdf/mobile_dual_arm.xacro (robot description, xacro)
@@ -1,58 +1,106 @@
 <?xml version="1.0"?>
 <robot name="mobile_dual_arm" xmlns:xacro="http://www.ros.org/wiki/xacro">
-	<xacro:include filename="$(find single_arm_description)/urdf/single_arm.xacro" />
-	<xacro:include filename="$(find Slide_rail)/urdf/Slide_rail.xacro" />
-	<xacro:include filename="$(find suction_urdf)/urdf/suction_urdf.xacro" />
-	<!--xacro:include filename="$(find single_arm_description)/urdf/materials.xacro" /-->
+  <xacro:include filename="$(find single_arm_description)/urdf/single_arm.xacro" />
+  <xacro:include filename="$(find Slide_rail)/urdf/Slide_rail.xacro" />
+  <xacro:include filename="$(find suction_urdf)/urdf/suction_urdf.xacro" />
+  <!--xacro:include filename="$(find single_arm_description)/urdf/materials.xacro" /-->
   <xacro:include filename="$(find mobile_dual_arm)/urdf/mobile_dual_arm.gazebo" />
   <xacro:include filename="$(find mobile_table)/urdf/mobile_table.xacro" />
-	<link name="world"/>
-	<!-- <joint name="fixed1" type="fixed">
-		<origin
-	    xyz="0 0 0.562"
+  <link name="world"/>
+  <!-- <joint name="fixed1" type="fixed">
+    <origin
+      xyz="0 0 0.562"
       rpy="0 0 0" />
-		<parent link="world"/>
+    <parent link="world"/>
     <child link="base_link"/>
-	</joint> -->
-	<joint name="fixed3" type="fixed">
-		<origin
-	    	xyz="0 0 0.562"
-        rpy="0 0 0" />
-		<parent link="world"/>
+  </joint> -->
+  <joint name="fixed3" type="fixed">
+    <origin
+      xyz="0 0 0.562"
+      rpy="0 0 0" />
+    <parent link="world"/>
     <child link="mobile_base"/>
-	</joint>
+  </joint>
   <xacro:single_arm side="r"  parent="Arm_Base_R_Link" child="r_tool_link">
-	  <origin xyz="0 -0.016 0" rpy="1.57 1.57 0" />
+    <origin xyz="0 -0.016 0" rpy="1.57 1.57 0" />
   </xacro:single_arm>
   <xacro:suction side="r"  parent="r_Link_6">
-	  <origin xyz="0 -0.016 0" rpy="0 0 0" />
+    <origin xyz="0 -0.016 0" rpy="0 0 0" />
   </xacro:suction>
   <xacro:single_arm side="l"  parent="Arm_Base_L_Link" child="l_tool_link">
-	  <origin xyz="0 0.016 0" rpy="-1.57 1.57 0" />
+    <origin xyz="0 0.016 0" rpy="-1.57 1.57 0" />
   </xacro:single_arm>
   <xacro:suction side="l"  parent="l_Link_6">
-	  <origin xyz="0 0.016 0" rpy="0 0 0" />
+    <origin xyz="0 0.016 0" rpy="0 0 0" />
   </xacro:suction>
-	<!--joint name="fixed" type="fixed">
-		<origin
-	    	xyz="0 0.016 0"
-        	rpy="-1.57 1.57 0" />
-		<parent link="Arm_Base_L_Link"/>
-     		<child link="Base"/>
-	</joint-->
-	<joint name="fixed1" type="fixed">
-		<origin
-	    xyz="0 0 0"
+  <!--joint name="fixed" type="fixed">
+    <origin
+      xyz="0 0.016 0"
+      rpy="-1.57 1.57 0" />
+    <parent link="Arm_Base_L_Link"/>
+    <child link="Base"/>
+  </joint-->
+  <joint name="fixed1" type="fixed">
+    <origin
+      xyz="0 0 0"
       rpy="0 0 0" />
-		<parent link="mobile_base"/>
+    <parent link="mobile_base"/>
     <child link="base_link"/>
-	</joint>
-	<!--joint name="fixed2" type="fixed">
-		<origin
-	    	xyz="0 -0.016 0"
-        	rpy="1.57 1.57 0" />
-		<parent link="Arm_Base_R_Link"/>
-     		<child link="Arm_Base_R"/>
-	</joint-->
+  </joint>
+  <!--joint name="fixed2" type="fixed">
+    <origin
+      xyz="0 -0.016 0"
+      rpy="1.57 1.57 0" />
+    <parent link="Arm_Base_R_Link"/>
+    <child link="Arm_Base_R"/>
+  </joint-->
+<link
+  name="Bin">
+    <inertial>
+      <origin
+	xyz="0 0 0"
+	rpy="0 0 0" />
+      <mass
+	value="0.823603974032196" />
+      <inertia
+	ixx="0"
+	ixy="0"
+	ixz="0"
+	iyy="0"
+	iyz="0"
+	izz="0" />
+    </inertial>
+    <visual>
+      <origin
+	xyz="0 0 0"
+	rpy="0 0 0" />
+      <geometry>
+	<mesh
+          scale="0.001 0.001 0.001"
+	  filename="package://mobile_dual_arm/scene/meshes/bin.STL" />
+      </geometry>
+      <material
+	name="blue_">
+	<color
+	  rgba="0.4 0.66 0.99 1" />
+      </material>
+    </visual>
+    <collision>
+      <origin
+	xyz="0 0 0"
+	rpy="0 0 0" />
+      <geometry>
+	<mesh
+	  filename="package://mobile_dual_arm/scene/meshes/bin.STL" />
+      </geometry>
+    </collision>
+  </link>
+  <joint name="fixed4" type="fixed">
+    <origin
+      xyz="-0.3 -0.31 0.06"
+      rpy="0 0 1.5708" />
+    <parent link="mobile_base"/>
+    <child link="Bin"/>
+  </joint>
   <!--transmission name="tran1">
     <type>transmission_interface/SimpleTransmission</type>

Commit message: Added New Object in to Gazebo Added Suction Control to Simulation

File: wrs_gazebo/mobile_dual_arm/urdf/mobile_dual_arm.xacro (robot description, xacro)
@@ -55,6 +55,5 @@
     <child link="Arm_Base_R"/>
   </joint-->
-<link
-  name="Bin">
+  <link name="Bin">
     <inertial>
       <origin
@@ -92,4 +91,5 @@
       <geometry>
 	<mesh
+          scale="0.001 0.001 0.001"
 	  filename="package://mobile_dual_arm/scene/meshes/bin.STL" />
       </geometry>
@@ -103,124 +103,4 @@
     <child link="Bin"/>
   </joint>
-  <!--transmission name="tran1">
-    <type>transmission_interface/SimpleTransmission</type>
-    <joint name="joint_1">
-      <hardwareInterface>hardware_interface/PositionJointInterface</hardwareInterface>
-    </joint>
-    <actuator name="motor1">
-      <hardwareInterface>hardware_interface/PositionJointInterface</hardwareInterface>
-      <mechanicalReduction>1</mechanicalReduction>
-    </actuator>
-  </transmission>
-  <transmission name="tran2">
-    <type>transmission_interface/SimpleTransmission</type>
-    <joint name="joint_2">
-      <hardwareInterface>hardware_interface/PositionJointInterface</hardwareInterface>
-    </joint>
-    <actuator name="motor2">
-      <hardwareInterface>hardware_interface/PositionJointInterface</hardwareInterface>
-      <mechanicalReduction>1</mechanicalReduction>
-    </actuator>
-  </transmission>
-  <transmission name="tran3">
-    <type>transmission_interface/SimpleTransmission</type>
-    <joint name="joint_3">
-      <hardwareInterface>hardware_interface/PositionJointInterface</hardwareInterface>
-    </joint>
-    <actuator name="motor3">
-      <hardwareInterface>hardware_interface/PositionJointInterface</hardwareInterface>
-      <mechanicalReduction>1</mechanicalReduction>
-    </actuator>
-  </transmission>
-  <transmission name="tran4">
-    <type>transmission_interface/SimpleTransmission</type>
-    <joint name="joint_4">
-      <hardwareInterface>hardware_interface/PositionJointInterface</hardwareInterface>
-    </joint>
-    <actuator name="motor4">
-      <hardwareInterface>hardware_interface/PositionJointInterface</hardwareInterface>
-      <mechanicalReduction>1</mechanicalReduction>
-    </actuator>
-  </transmission>
-  <transmission name="tran5">
-    <type>transmission_interface/SimpleTransmission</type>
-    <joint name="joint_5">
-      <hardwareInterface>hardware_interface/PositionJointInterface</hardwareInterface>
-    </joint>
-    <actuator name="motor5">
-      <hardwareInterface>hardware_interface/PositionJointInterface</hardwareInterface>
-      <mechanicalReduction>1</mechanicalReduction>
-    </actuator>
-  </transmission>
-  <transmission name="tran6">
-    <type>transmission_interface/SimpleTransmission</type>
-    <joint name="joint_6">
-      <hardwareInterface>hardware_interface/PositionJointInterface</hardwareInterface>
-    </joint>
-    <actuator name="motor6">
-      <hardwareInterface>hardware_interface/PositionJointInterface</hardwareInterface>
-      <mechanicalReduction>1</mechanicalReduction>
-    </actuator>
-  </transmission>
-  <transmission name="tran1_R">
-    <type>transmission_interface/SimpleTransmission</type>
-    <joint name="joint_R_1">
-      <hardwareInterface>hardware_interface/PositionJointInterface</hardwareInterface>
-    </joint>
-    <actuator name="motor1_R">
-      <hardwareInterface>hardware_interface/PositionJointInterface</hardwareInterface>
-      <mechanicalReduction>1</mechanicalReduction>
-    </actuator>
-  </transmission>
-  <transmission name="tran2_R">
-    <type>transmission_interface/SimpleTransmission</type>
-    <joint name="joint_R_2">
-      <hardwareInterface>hardware_interface/PositionJointInterface</hardwareInterface>
-    </joint>
-    <actuator name="motor2_R">
-      <hardwareInterface>hardware_interface/PositionJointInterface</hardwareInterface>
-      <mechanicalReduction>1</mechanicalReduction>
-    </actuator>
-  </transmission>
-  <transmission name="tran3_R">
-    <type>transmission_interface/SimpleTransmission</type>
-    <joint name="joint_R_3">
-      <hardwareInterface>hardware_interface/PositionJointInterface</hardwareInterface>
-    </joint>
-    <actuator name="motor3_R">
-      <hardwareInterface>hardware_interface/PositionJointInterface</hardwareInterface>
-      <mechanicalReduction>1</mechanicalReduction>
-    </actuator>
-  </transmission>
-  <transmission name="tran4_R">
-    <type>transmission_interface/SimpleTransmission</type>
-    <joint name="joint_R_4">
-      <hardwareInterface>hardware_interface/PositionJointInterface</hardwareInterface>
-    </joint>
-    <actuator name="motor4_R">s
-      <hardwareInterface>hardware_interface/PositionJointInterface</hardwareInterface>
-      <mechanicalReduction>1</mechanicalReduction>
-    </actuator>
-  </transmission>
-  <transmission name="tran5_R">
-    <type>transmission_interface/SimpleTransmission</type>
-    <joint name="joint_R_5">
-      <hardwareInterface>hardware_interface/PositionJointInterface</hardwareInterface>
-    </joint>
-    <actuator name="motor5_R">
-      <hardwareInterface>hardware_interface/PositionJointInterface</hardwareInterface>
-      <mechanicalReduction>1</mechanicalReduction>
-    </actuator>
-  </transmission>
-  <transmission name="tran6_R">
-    <type>transmission_interface/SimpleTransmission</type>
-    <joint name="joint_R_6">
-      <hardwareInterface>hardware_interface/PositionJointInterface</hardwareInterface>
-    </joint>
-    <actuator name="motor6_R">
-      <hardwareInterface>hardware_interface/PositionJointInterface</hardwareInterface>
-      <mechanicalReduction>1</mechanicalReduction>
-    </actuator>
-  </transmission-->
   <transmission name="tran1_slide_R">
     <type>transmission_interface/SimpleTransmission</type>
