Commit message: Change Euler Angle Define

File: wrs_gazebo/single_arm/single_arm_description/urdf/single_arm.xacro (robot description, xacro)
@@ -5,5 +5,5 @@
   <xacro:include filename="$(find single_arm_description)/urdf/materials.xacro" />
   <!-- Constants for robot dimensions -->
-  <xacro:macro name="single_arm" params="side parent child *origin">
+  <xacro:macro name="single_arm" params="side parent child toolrot *origin">
 	  <link
 	    name="${side}_Base">
@@ -439,22 +439,22 @@
 	    </collision>
 	  </link> -->
-	  <joint
-	    name="${side}_joint_7"
-	    type="revolute">
-	    <origin
-	      xyz="0 -0.1345 0"
-	      rpy="1.5708 4.5659E-16 1.2025E-31" />
-	    <parent
-	      link="${side}_Link_6" />
-	    <child
-	      link="${child}" />
-	    <axis
-	      xyz="0 0 1" />
-	    <limit
-	      lower="-3.14"
-	      upper="3.14"
-	      effort="22"
-	      velocity="65" />
-	  </joint>
+		<joint
+			name="${side}_joint_7"
+			type="revolute">
+			<origin
+				xyz="0 -0.1345 0"
+				rpy="1.5708 ${toolrot} 0" />
+			<parent
+				link="${side}_Link_6" />
+			<child
+				link="${child}" />
+			<axis
+				xyz="0 0 1" />
+			<limit
+				lower="-3.14"
+				upper="3.14"
+				effort="22"
+				velocity="65" />
+		</joint>
           <!--
 	  <link
